Commit message: joint axis testing

File: Week 8/ros2_ws/install/ros2_path_planning/share/ros2_path_planning/urdf/maze_bot.urdf (robot description, URDF)
Before this commit: robot maze_bot, 5 links, 4 joints
Links:
- link base: geometry collision mesh filename=package://ros2_path_planning/meshes/Base.stl; visual mesh filename=package://ros2_path_planning/meshes/Base.stl
Joints:
- joint base_joint: origin xyz=0.0 0.0 0.0 rpy=0.0 0.0 0.005 -> xyz=0.0 0.0 0.03 rpy=0.0 0.0 0.0
- joint caster_joint: origin xyz=0.0 0.0 0.0 rpy=0.0 0.0 0.0 -> xyz=-0.035 0.0 -0.017 rpy=0.0 0.0 0.0
- joint wheel_left_joint: origin xyz=0.0 0.0 0.0 rpy=0.0 0.0 0.0 -> xyz=0.02 -0.03 0.0 rpy=0.0 0.0 0.0
- joint wheel_right_joint: origin xyz=0.0 0.0 0.0 rpy=0.0 0.0 0.0 -> xyz=0.02 0.024 0.0 rpy=0.0 0.0 0.0

File: Week 8/ros2_ws/src/ros2_path_planning/urdf/maze_bot.urdf (robot description, URDF)
Before this commit: robot maze_bot, 5 links, 4 joints
Links:
- link base: geometry collision mesh filename=package://ros2_path_planning/meshes/Base.stl; visual mesh filename=package://ros2_path_planning/meshes/Base.stl
Joints:
- joint base_joint: origin xyz=0.0 0.0 0.0 rpy=0.0 0.0 0.005 -> xyz=0.0 0.0 0.03 rpy=0.0 0.0 0.0
- joint caster_joint: origin xyz=0.0 0.0 0.0 rpy=0.0 0.0 0.0 -> xyz=-0.035 0.0 -0.017 rpy=0.0 0.0 0.0
- joint wheel_left_joint: origin xyz=0.0 0.0 0.0 rpy=0.0 0.0 0.0 -> xyz=0.02 -0.03 0.0 rpy=0.0 0.0 0.0
- joint wheel_right_joint: origin xyz=0.0 0.0 0.0 rpy=0.0 0.0 0.0 -> xyz=0.02 0.024 0.0 rpy=0.0 0.0 0.0
